Commit message: 27/04/2026

File: puzzlebot_description/urdf/mcr2_control/gazebo_control.xacro (robot description, xacro)
@@ -3,61 +3,25 @@
 <xacro:macro name="puzzlebot_control" params="prefix">
     <gazebo>
-        <!--<plugin name="DiffDynamicPlugin" filename="libDiffDynamicPlugin.so">
-                <leftJoint>${prefix}wheel_left_joint</leftJoint>
-                <rightJoint>${prefix}wheel_right_joint</rightJoint>
-                <cmd_R_topic>${prefix}VelocitySetR</cmd_R_topic>
-                <cmd_L_topic>${prefix}VelocitySetL</cmd_L_topic>
-                <cmd_vel_topic>${prefix}cmd_vel</cmd_vel_topic>
-                <enc_R_topic>${prefix}VelocityEncR</enc_R_topic>
-                <enc_L_topic>${prefix}VelocityEncL</enc_L_topic>
-                <robot_vel_topic>${prefix}robot_vel</robot_vel_topic>
-                <mot_Vmax>5</mot_Vmax>
-                <mot_J>0.0005</mot_J>
-                <mot_R>2</mot_R>
-                <mot_L>0.01</mot_L>
-                <mot_K>0.01</mot_K>
-                <mot_b>0.00001</mot_b>
-                <mot_gear>34</mot_gear>
-                <robot_width>0.19</robot_width>
-                <wheel_radius>0.05</wheel_radius>
-                <pid_Kp>0.1</pid_Kp>
-                <pid_Ti>0.05</pid_Ti>
-                <pid_Td>0</pid_Td>
-                <input_type>1</input_type>
-                <rate>100</rate>
-        </plugin>-->
-        <plugin filename="gz-sim-diff-drive-system" name="gz::sim::systems::DiffDrive">
-            <odom_publisher_frequency>50</odom_publisher_frequency>
+        <plugin name="gazebo_ros_diff_drive" filename="libgazebo_ros_diff_drive.so">
+            <update_rate>50</update_rate>
             <left_joint>${prefix}wheel_left_joint</left_joint>
             <right_joint>${prefix}wheel_right_joint</right_joint>
             <wheel_separation>0.19</wheel_separation>
-            <wheel_radius>0.05</wheel_radius>
-            <topic>cmd_vel</topic>
-            <tf_topic>tf</tf_topic>
-            <odom_topic>odom</odom_topic>
-            <frame_id>odom</frame_id>
-            <child_frame_id>base_footprint</child_frame_id>
-            <max_angular_acceleration>1.8</max_angular_acceleration>
-            <max_angular_velocity>13.0</max_angular_velocity>
+            <wheel_diameter>0.10</wheel_diameter>
+            <max_wheel_torque>20</max_wheel_torque>
+            <max_wheel_acceleration>1.0</max_wheel_acceleration>
+            <command_topic>cmd_vel</command_topic>
+            <odometry_topic>odom</odometry_topic>
+            <odometry_frame>odom</odometry_frame>
+            <robot_base_frame>${prefix}base_footprint</robot_base_frame>
+            <publish_odom>true</publish_odom>
+            <publish_odom_tf>true</publish_odom_tf>
+            <publish_wheel_tf>false</publish_wheel_tf>
         </plugin>
-        <plugin filename="gz-sim-joint-state-publisher-system" name="gz::sim::systems::JointStatePublisher">
-            <topic>${prefix}joint_states</topic>
+        <plugin name="gazebo_ros_joint_state_publisher" filename="libgazebo_ros_joint_state_publisher.so">
             <update_rate>50</update_rate>
             <joint_name>${prefix}wheel_right_joint</joint_name>
             <joint_name>${prefix}wheel_left_joint</joint_name>
         </plugin>
-        <plugin
-                filename="gz-sim-sensors-system"
-                name="gz::sim::systems::Sensors">
-                <render_engine>ogre2</render_engine>
-        </plugin>
-        <!--<plugin filename="gz-sim-odometry-publisher-system" name="gz::sim::systems::OdometryPublisher">
-        <odom_frame>world</odom_frame>
-        <robot_base_frame>${prefix}base_footprint</robot_base_frame>
-        <odom_publish_frequency>50</odom_publish_frequency>
-        <odom_topic>${prefix}ground_truth</odom_topic>
-        <tf_topic>tf</tf_topic>
-        <dimensions>2</dimensions>
-        </plugin>-->
     </gazebo>
 </xacro:macro>

File: puzzlebot_description/urdf/mcr2_sensors/lidar.xacro (robot description, xacro)
@@ -55,14 +55,10 @@
         <visual>
             <origin xyz="${lidar_base_mesh_pos_x} ${lidar_base_mesh_pos_y} ${lidar_base_mesh_pos_z}" rpy="${lidar_base_mesh_pos_r} ${lidar_base_mesh_pos_p} ${lidar_base_mesh_pos_w}"/>
-            <geometry>
-                <mesh filename="${mesh_file}"/>
-            </geometry>
+            <geometry><mesh filename="${mesh_file}"/></geometry>
             <material name="grey"/>
         </visual>
         <collision>
             <origin xyz="${lidar_base_collision_pos_x} ${lidar_base_collision_pos_y} ${lidar_base_collision_pos_z}" rpy="${lidar_base_collision_pos_r} ${lidar_base_collision_pos_p} ${lidar_base_collision_pos_w}"/>
-            <geometry>
-                <box size="${lidar_base_length} ${lidar_base_width} ${lidar_base_height}"/>
-            </geometry>
+            <geometry><box size="${lidar_base_length} ${lidar_base_width} ${lidar_base_height}"/></geometry>
         </collision>
         <inertial>
@@ -75,14 +71,10 @@
         <visual>
             <origin xyz="0 0 0" rpy="0 0 0"/>
-            <geometry>
-                <box size="0.005 0.005 0.005"/> <!-- Box shape for lidar -->
-            </geometry>
+            <geometry><box size="0.005 0.005 0.005"/></geometry>
             <material name="grey"/>
         </visual>
         <collision>
             <origin xyz="0 0 0" rpy="0 0 0"/>
-            <geometry>
-                <box size="0.005 0.005 0.005"/>
-            </geometry>
+            <geometry><box size="0.005 0.005 0.005"/></geometry>
         </collision>
         <inertial>
@@ -102,41 +94,34 @@
         <origin xyz="${lidar_pos_x} ${lidar_pos_y} ${lidar_pos_z}" rpy="${lidar_pos_r} ${lidar_pos_p} ${lidar_pos_w}"/>
     </joint>
-    <!--<gazebo reference='${prefix}lidar_base_joint'>
-    <preserveFixedJoint>true</preserveFixedJoint>
-    </gazebo>
-    <gazebo reference='${prefix}lidar_joint'>
-    <preserveFixedJoint>true</preserveFixedJoint>
-    </gazebo>-->
     <gazebo reference="${prefix}laser_frame">
-        <sensor name="${prefix}lidar_sensor" type="gpu_lidar">
-            <topic>${prefix}${topic_name}</topic>
-            <gz_frame_id>${prefix}laser_frame</gz_frame_id>
-            <pose> 0 0 0 0 0 0 </pose>
+        <sensor name="${prefix}lidar_sensor" type="ray">
+            <pose>0 0 0 0 0 0</pose>
             <update_rate>${update_rate}</update_rate>
             <always_on>${always_on}</always_on>
             <visualize>${visualize}</visualize>
             <ray>
-            <scan>
-                <horizontal>
-                <samples>${ray_count}</samples>
-                <resolution>1</resolution>
-                <min_angle>${min_angle}</min_angle>
-                <max_angle>${max_angle}</max_angle>
-                </horizontal>
-                <vertical>
-                <samples>1</samples>
-                <resolution>0.01</resolution>
-                <min_angle>0</min_angle>
-                <max_angle>0</max_angle>
-                </vertical>
-            </scan>
-            <range>
-                <min>${min_range}</min>
-                <max>${max_range}</max>
-                <resolution>${range_resolution}</resolution>
-            </range>
+                <scan>
+                    <horizontal>
+                        <samples>${ray_count}</samples>
+                        <resolution>1</resolution>
+                        <min_angle>${min_angle}</min_angle>
+                        <max_angle>${max_angle}</max_angle>
+                    </horizontal>
+                </scan>
+                <range>
+                    <min>${min_range}</min>
+                    <max>${max_range}</max>
+                    <resolution>${range_resolution}</resolution>
+                </range>
             </ray>
+            <plugin name="gazebo_ros_lidar" filename="libgazebo_ros_ray_sensor.so">
+                <ros>
+                    <remapping>~/out:=${topic_name}</remapping>
+                </ros>
+                <output_type>sensor_msgs/LaserScan</output_type>
+                <frame_name>${prefix}laser_frame</frame_name>
+            </plugin>
         </sensor>
     </gazebo>
-    </xacro:macro>
+  </xacro:macro>
 </robot>
